File: hw/boards/bms/leak_sensing.kicad_sch (KiCad schematic)
At the start: 0 parts

Commit message: leak_sensing component
Parts:
- added D1: LED, symbol Device:LED
- added J1, J2, J3, J4, J5: Conn_01x02, symbol Connector_Generic:Conn_01x02
- added Q1: Q_PMOS_GDS, Package_TO_SOT_SMD:TO-252-2, symbol Transistor_FET:Q_PMOS_GDS
- added R1, R3, R4: 1k, Package_TO_SOT_SMD:TO-252-2, symbol Device:R_US
- added R2: 27k, Package_TO_SOT_SMD:TO-252-2, symbol Device:R_US
- added TP1, TP2, TP3: TestPoint, symbol Connector:TestPoint
Connections:
- new net: D1.2 (A), R4.2
- new net: Q1.1 (G), R1.2, R2.2
- new net +3V3: Q1.2 (D), R2.1
- new net GND: D1.1 (K), J1.1 (Pin_1), J2.1 (Pin_1), J3.1 (Pin_1), J4.1 (Pin_1), J5.1 (Pin_1), R3.2
- new net LEAK_SIGNAL: Q1.3 (S), R3.1, R4.1, TP3.1
- new net PROBE: J1.2 (Pin_2), J2.2 (Pin_2), J3.2 (Pin_2), J4.2 (Pin_2), J5.2 (Pin_2), R1.1, TP1.1, TP2.1
Other:
- note added: "https://bluerobotics.com/wp-content/uploads/2018/10/SOS-LEAK-SENSOR-SCHEMATIC.pdf"
