File: hw/boards/bms/cell_monitoring.kicad_sch (KiCad schematic)
At the start: 0 parts

Commit message: Added Cell Monitoring
Parts:
- added C10, C3, C4, C5, C6, C7, C8, C9: 10nF, symbol Device:C
- added D10, D11, D4, D5, D6, D7, D8, D9: 3.3V, symbol Device:D_Zener
- added J7, J8: Conn_01x05_Pin, Connector_JST:JST_XH_B5B-XH-AM_1x05_P2.50mm_Vertical, symbol Connector:Conn_01x05_Pin
- added R10, R16: 44.2k, symbol Device:R_US
- added R11, R17: 18.7k, symbol Device:R_US
- added R12, R15, R18, R23, R24, R29, R30, R9: 1k, symbol Device:R_US
- added R13, R7: 45.3k, symbol Device:R_US
- added R14, R8: 13k, symbol Device:R_US
- added R19, R21: 20.5k, symbol Device:R_US
- added R20, R22: 16.5k, symbol Device:R_US
- added R25, R27: 10k, symbol Device:R_US
- added R26, R28: 82.5k, symbol Device:R_US
Connections:
- new net: C7.1, R19.2, R20.1, R23.1
- new net: C3.1, R7.2, R8.1, R9.1
- new net: C4.1, R10.2, R11.1, R12.1
- new net: C6.1, R16.2, R17.1, R18.1
- new net: C8.1, R21.2, R22.1, R24.1
- new net: C5.1, R13.2, R14.1, R15.1
- new net: C9.1, R25.2, R26.1, R29.1
- new net: C10.1, R27.2, R28.1, R30.1
- new net 11.1V (1): J7.2 (Pin_2), R10.1
- new net 11.1V (2): J8.2 (Pin_2), R16.1
- new net 14.8V (1): J7.1 (Pin_1), R7.1
- new net 14.8V (2): J8.1 (Pin_1), R13.1
- new net 3.7V (1): J7.4 (Pin_4), R25.1
- new net 3.7V (2): J8.4 (Pin_4), R27.1
- new net 7.4V (1): J7.3 (Pin_3), R19.1
- new net 7.4V (2): J8.3 (Pin_3), R21.1
- new net GND: C10.2, C3.2, C4.2, C5.2, C6.2, C7.2, C8.2, C9.2, D10.2 (A), D11.2 (A), D4.2 (A), D5.2 (A), D6.2 (A), D7.2 (A), D8.2 (A), D9.2 (A), J7.5 (Pin_5), J8.5 (Pin_5), R11.2, R14.2, R17.2, R20.2, R22.2, R26.2, R28.2, R8.2
- new net OUT1: D4.1 (K), R9.2
- new net OUT2: D6.1 (K), R12.2
- new net OUT3: D8.1 (K), R23.2
- new net OUT4: D10.1 (K), R29.2
- new net OUT5: D5.1 (K), R15.2
- new net OUT6: D7.1 (K), R18.2
- new net OUT7: D9.1 (K), R24.2
- new net OUT8: D11.1 (K), R30.2
