File: hw/boards/bms/thermal_monitoring.kicad_sch (KiCad schematic)
At the start: 0 parts

Commit message: thermal monitoring + project file resolve
Parts:
- added C1: 0.01u, symbol Device:C
- added C2: 10u, symbol Device:C
- added D1, D2: D, symbol Device:D
- added FB1, FB2: Ferrite, symbol Device:FerriteBead_Small
- added J1: Thermocouple IN, symbol Connector_Generic:Conn_01x02
- added R1, R2: 10k, symbol Device:R_US
- added U1: MAX31855KASA, Package_SO:SOIC-8_3.9x4.9mm_P1.27mm, symbol Sensor_Temperature:MAX31855KASA
Connections:
- new net: D2.2 (A), R2.1, U1.6 (~{CS})
- new net: FB2.1, J1.2 (Pin_2)
- new net: C1.2, FB2.2, U1.2 (T-)
- new net: D1.2 (A), R1.2, U1.5 (SCK)
- new net: C1.1, FB1.2, U1.3 (T+)
- new net: FB1.1, J1.1 (Pin_1)
- new net +3.3V: C2.1, R1.1, R2.2, U1.4 (V_{CC})
- new net GND: C2.2, U1.1 (GND)
- new net cs: D2.1 (K)
- new net sck: D1.1 (K)
- new net so: U1.7 (SO)
